File: hw/sch_pcb/OLED02.kicad_pcb (KiCad board)
At the start: 2 copper layers, 40.1 x 40.1 mm, 23 parts, among them J2 HEADER_2x05_PARALLEL, M1 HOLE, M2 HOLE, M3 HOLE, M4 HOLE

Commit message: update kicad version
Parts:
- added C9: 4u7, Capacitor_SMD:C_0805_2012Metric, B.Cu at (132.5, 103.2)
- moved D2 2.98 mm to (142.4, 113.7)
- moved R1 0.07 mm to (136.4, 103.2)
Connections:
- DS1 pad 12: unconnected-(DS1-BS2-Pad12) -> GND
- DS1 pad 16: unconnected-(DS1-R/~{W}-Pad16) -> GND
- DS1 pad 17: unconnected-(DS1-E/~{RD}-Pad17) -> GND
- DS1 pad 21: unconnected-(DS1-D3-Pad21) -> GND
- DS1 pad 22: unconnected-(DS1-D4-Pad22) -> GND
- DS1 pad 23: unconnected-(DS1-D5-Pad23) -> GND
- DS1 pad 24: unconnected-(DS1-D6-Pad24) -> GND
- DS1 pad 25: unconnected-(DS1-D7-Pad25) -> GND
- DS1 pad 28: +3.3V -> Net-(DS1-VCC)
Routing:
- net GND: track 28.6 -> 44.0 mm, vias 42 -> 45
- net Net-(DS1-VCC): track 0.00 -> 4.63 mm
- net +3.3V: track 113.6 -> 110.3 mm
Other:
- board text added: "0x3C 0x3D"
- board text added: "0x3D 0x3C"
- board text added: "Fix addr 0x3C"
- board text removed: "0x77/0x78"
- board text removed: "Fix addr"
